File: clock.kicad_pcb (KiCad board)
At the start: 2 copper layers, 160 x 100 mm, 44 parts, among them CON201 BARREL_JACK, P201 CONN_01X05, P701 CONN_01X06, SW301 Coded_Switch, SW302 Coded_Switch, SW401 Coded_Switch, SW402 Coded_Switch, SW601 SW_PUSH_SMALL_H, SW602 SW_PUSH_SMALL_H, U101 4011, U301 74LS47, U302 4510, U303 74LS47, U304 4510, U305 4538, U306 74LS688, U307 74LS688, U401 74LS47, U402 4510, U403 74LS47, U404 4510, U405 74LS688, U406 74LS688, U501 74LS47, U502 4510, U503 74LS47, U504 4510, U505 4538, U506 74LS688, U601 arduino_mini, U602 4017

Commit message: some revisions
Parts:
- removed P701: CONN_01X06, Pin_Headers:Pin_Header_Straight_1x06
- removed SW601: SW_PUSH_SMALL_H, Buttons_Switches_ThroughHole:SW_PUSH_SMALL
- removed U501, U503: 74LS47, Housings_DIP:DIP-16_W7.62mm
- removed U506: 74LS688, Housings_DIP:DIP-20_W7.62mm
- added D701: Diode_Bridge, w_pth_diodes:bridge_wob, F.Cu at (0.00, 0.00)
- added P202, P203, P301, P302, P402, P403: CONN_01X07, Pin_Headers:Pin_Header_Straight_1x07, F.Cu at (0.00, 0.00)
- added P401, P501: CONN_01X09, Pin_Headers:Pin_Header_Straight_1x09, F.Cu at (0.00, 0.00)
- added R502: 10k, Resistors_ThroughHole:Resistor_Horizontal_RM10mm, F.Cu at (0.00, 0.00)
- added R701: 15k, Resistors_ThroughHole:Resistor_Horizontal_RM10mm, F.Cu at (0.00, 0.00)
- added SW501: SPST, Pin_Headers:Pin_Header_Straight_1x02, F.Cu at (0.00, 0.00)
- added U201, U202: 4511, Housings_DIP:DIP-16_W7.62mm, F.Cu at (0.00, 0.00)
- added U603, U604: 4017, Housings_DIP:DIP-16_W7.62mm, F.Cu at (0.00, 0.00)
- U301, U303, U403: value 74LS47 -> 4511
- U401: value 74LS47 -> 4011; footprint Housings_DIP:DIP-16_W7.62mm -> Housings_DIP:DIP-14_W7.62mm
- U406: value 74LS688 -> 4511; footprint Housings_DIP:DIP-20_W7.62mm -> Housings_DIP:DIP-16_W7.62mm
- moved U303 260.8 mm to (0.00, 0.00), turned to 0 degrees
- moved U301 238.1 mm to (0.00, 0.00), turned to 0 degrees
- moved D201 220.5 mm to (0.00, 0.00)
- moved D202 220.5 mm to (0.00, 0.00)
- moved D203 220.5 mm to (0.00, 0.00)
- moved D204 220.5 mm to (0.00, 0.00)
- moved P201 220.5 mm to (0.00, 0.00)
- moved U406 220.5 mm to (0.00, 0.00)
- moved U403 216.1 mm to (0.00, 0.00), turned to 0 degrees
- moved U401 195.1 mm to (0.00, 0.00), turned to 0 degrees
- moved CON201 128.4 mm to (0.00, 0.00), turned to 0 degrees
- moved U101 126.2 mm to (0.00, 0.00)
Connections:
- CON201 pad 1: +9V -> Net-(CON201-Pad1)
- CON201 pad 2: GND -> Net-(CON201-Pad2)
- CON201 pad 3: GND -> Net-(CON201-Pad2)
- U101 pad 10: (no net) -> /Hours/CIN
- U101 pad 14: VDD -> +5V
- U101 pad 7: VSS -> GND
- U101 pad 8: (no net) -> Net-(P401-Pad7)
- U101 pad 9: (no net) -> Net-(P401-Pad8)
- U301 pad 1: Net-(U301-Pad1) -> Net-(P401-Pad3)
- U301 pad 16: VCC -> +5V
- U301 pad 2: Net-(U301-Pad2) -> Net-(P401-Pad4)
- U301 pad 3: (no net) -> +5V
- U301 pad 4: (no net) -> +5V
- U301 pad 5: (no net) -> GND
- U301 pad 6: Net-(U301-Pad6) -> Net-(P401-Pad5)
- U301 pad 7: Net-(U301-Pad7) -> Net-(P401-Pad2)
- U302 pad 11: Net-(U301-Pad1) -> Net-(U201-Pad1)
- U302 pad 14: Net-(U301-Pad2) -> Net-(U201-Pad2)
- U302 pad 15: /Hours/CLK -> /Hours/CIN
- U302 pad 16: VDD -> +5V
- U302 pad 2: Net-(U301-Pad6) -> Net-(U201-Pad6)
- U302 pad 5: /Hours/CIN -> GND
- U302 pad 6: Net-(U301-Pad7) -> Net-(U201-Pad7)
- U302 pad 8: VSS -> GND
- U303 pad 1: Net-(U303-Pad1) -> Net-(P401-Pad7)
- U303 pad 16: VCC -> +5V
- U303 pad 2: Net-(U303-Pad2) -> Net-(P401-Pad8)
- U303 pad 3: (no net) -> +5V
- U303 pad 4: (no net) -> +5V
- U303 pad 5: (no net) -> GND
- U303 pad 6: Net-(U303-Pad6) -> Net-(P401-Pad9)
- U303 pad 7: Net-(U303-Pad7) -> Net-(P401-Pad6)
- U304 pad 11: Net-(U303-Pad1) -> Net-(U202-Pad1)
- U304 pad 14: Net-(U303-Pad2) -> Net-(U202-Pad2)
- U304 pad 15: /Hours/CLK -> Net-(U302-Pad7)
- U304 pad 16: VDD -> +5V
- U304 pad 2: Net-(U303-Pad6) -> Net-(U202-Pad6)
- U304 pad 5: Net-(U302-Pad7) -> GND
- U304 pad 6: Net-(U303-Pad7) -> Net-(U202-Pad7)
- U304 pad 8: VSS -> GND
- U305 pad 16: VDD -> +5V
- U305 pad 8: VSS -> GND
- U306 pad 11: Net-(U303-Pad7) -> Net-(U202-Pad7)
- U306 pad 13: Net-(U303-Pad1) -> Net-(U202-Pad1)
- U306 pad 15: Net-(U303-Pad2) -> Net-(U202-Pad2)
- U306 pad 17: Net-(U303-Pad6) -> Net-(U202-Pad6)
- U306 pad 2: Net-(U301-Pad7) -> Net-(U201-Pad7)
- U306 pad 20: VCC -> +5V
- U306 pad 4: Net-(U301-Pad1) -> Net-(U201-Pad1)
- U306 pad 6: Net-(U301-Pad2) -> Net-(U201-Pad2)
- U306 pad 8: Net-(U301-Pad6) -> Net-(U201-Pad6)
- U307 pad 11: Net-(U303-Pad7) -> Net-(U202-Pad7)
- U307 pad 13: Net-(U303-Pad1) -> Net-(U202-Pad1)
- U307 pad 15: Net-(U303-Pad2) -> Net-(U202-Pad2)
- U307 pad 17: Net-(U303-Pad6) -> Net-(U202-Pad6)
- U307 pad 2: Net-(U301-Pad7) -> Net-(U201-Pad7)
- U307 pad 20: VCC -> +5V
- U307 pad 4: Net-(U301-Pad1) -> Net-(U201-Pad1)
- U307 pad 6: Net-(U301-Pad2) -> Net-(U201-Pad2)
- U307 pad 8: Net-(U301-Pad6) -> Net-(U201-Pad6)
- U401 pad 1: Net-(U401-Pad1) -> Net-(P501-Pad7)
- U401 pad 10: Net-(P401-Pad6) -> (no net)
- U401 pad 11: Net-(P401-Pad5) -> (no net)
- U401 pad 12: Net-(P401-Pad4) -> (no net)
- U401 pad 13: Net-(P401-Pad3) -> (no net)
- U401 pad 14: Net-(P401-Pad9) -> +5V
- U401 pad 2: Net-(U401-Pad2) -> Net-(P501-Pad8)
- U401 pad 3: (no net) -> /Minutes/CIN
- U401 pad 6: Net-(U401-Pad6) -> (no net)
- U401 pad 7: Net-(U401-Pad7) -> GND
- U401 pad 8: GND -> (no net)
- U401 pad 9: Net-(P401-Pad7) -> (no net)
- U402 pad 11: Net-(U401-Pad1) -> Net-(P401-Pad3)
- U402 pad 14: Net-(U401-Pad2) -> Net-(P401-Pad4)
- U402 pad 15: /Hours/CLK -> /Minutes/CIN
- U402 pad 16: VDD -> +5V
- U402 pad 2: Net-(U401-Pad6) -> Net-(P401-Pad5)
- U402 pad 5: /Minutes/CIN -> GND
- U402 pad 6: Net-(U401-Pad7) -> Net-(P401-Pad2)
- U402 pad 8: VSS -> GND
- U403 pad 1: Net-(U403-Pad1) -> Net-(P501-Pad3)
- U403 pad 16: VCC -> +5V
- U403 pad 2: Net-(U403-Pad2) -> Net-(P501-Pad4)
- U403 pad 3: (no net) -> +5V
- U403 pad 4: (no net) -> +5V
- U403 pad 5: (no net) -> GND
- U403 pad 6: Net-(U403-Pad6) -> Net-(P501-Pad5)
- U403 pad 7: Net-(U403-Pad7) -> Net-(P501-Pad2)
- U404 pad 11: Net-(U403-Pad1) -> Net-(P401-Pad7)
- U404 pad 14: Net-(U403-Pad2) -> Net-(P401-Pad8)
- U404 pad 15: /Hours/CLK -> Net-(U402-Pad7)
- U404 pad 16: VDD -> +5V
- U404 pad 2: Net-(U403-Pad6) -> Net-(P401-Pad9)
- U404 pad 5: Net-(U402-Pad7) -> GND
- U404 pad 6: Net-(U403-Pad7) -> Net-(P401-Pad6)
- U404 pad 8: VSS -> GND
- U405 pad 11: Net-(U403-Pad7) -> Net-(P401-Pad6)
- U405 pad 13: Net-(U403-Pad1) -> Net-(P401-Pad7)
- U405 pad 15: Net-(U403-Pad2) -> Net-(P401-Pad8)
- U405 pad 17: Net-(U403-Pad6) -> Net-(P401-Pad9)
- U405 pad 2: Net-(U401-Pad7) -> Net-(P401-Pad2)
- U405 pad 20: VCC -> +5V
- U405 pad 4: Net-(U401-Pad1) -> Net-(P401-Pad3)
- U405 pad 6: Net-(U401-Pad2) -> Net-(P401-Pad4)
- U405 pad 8: Net-(U401-Pad6) -> Net-(P401-Pad5)
- U406 pad 1: GND -> Net-(P501-Pad7)
- U406 pad 10: GND -> Net-(P403-Pad4)
- U406 pad 11: Net-(U403-Pad7) -> Net-(P403-Pad3)
- U406 pad 12: GND -> Net-(P403-Pad2)
- U406 pad 13: Net-(U403-Pad1) -> Net-(P403-Pad1)
- U406 pad 14: +5V -> Net-(P403-Pad7)
- U406 pad 15: Net-(U403-Pad2) -> Net-(P403-Pad6)
- U406 pad 2: Net-(U401-Pad7) -> Net-(P501-Pad8)
- U406 pad 3: GND -> +5V
- U406 pad 4: Net-(U401-Pad1) -> +5V
- U406 pad 6: Net-(U401-Pad2) -> (no net)
- U406 pad 7: GND -> Net-(P501-Pad6)
- U406 pad 8: Net-(U401-Pad6) -> GND
- U406 pad 9: GND -> Net-(P403-Pad5)
- U502 pad 11: Net-(U501-Pad1) -> Net-(P501-Pad3)
- U502 pad 14: Net-(U501-Pad2) -> Net-(P501-Pad4)
- U502 pad 15: /Hours/CLK -> /Seconds/CIN
- U502 pad 16: VDD -> +5V
- U502 pad 2: Net-(U501-Pad6) -> Net-(P501-Pad5)
- U502 pad 6: Net-(U501-Pad7) -> Net-(P501-Pad2)
- U502 pad 8: VSS -> GND
- U504 pad 11: Net-(U503-Pad1) -> Net-(P501-Pad7)
- U504 pad 14: Net-(U503-Pad2) -> Net-(P501-Pad8)
- U504 pad 15: /Hours/CLK -> Net-(U502-Pad7)
- U504 pad 16: VDD -> +5V
- U504 pad 5: Net-(U502-Pad7) -> GND
- U504 pad 6: Net-(U503-Pad7) -> Net-(P501-Pad6)
- U504 pad 8: VSS -> GND
- U505 pad 16: VDD -> +5V
- U505 pad 8: VSS -> GND
- U601 pad 21: Net-(SW601-Pad1) -> /Hours/COUT
- U601 pad 8: SDA -> (no net)
- U601 pad 9: SCL -> (no net)
- U602 pad 13: VSS -> GND
- U602 pad 16: VDD -> +5V
- U602 pad 8: VSS -> GND
